Commit message: updated README.md & urdf

File: kitchen_bot_description/urdf/kitchen_bot.urdf.xacro (robot description, xacro)
@@ -155,4 +155,40 @@
     <xacro:caster_wheel locationprefix="bl" locationright="-1" wheel_base_dx="${-kitchen_bot_back_caster_wheel_base_dx + kitchen_bot_act_wheel_dx}"/>
     <xacro:caster_wheel locationprefix="br" locationright="1" wheel_base_dx="${-kitchen_bot_back_caster_wheel_base_dx + kitchen_bot_act_wheel_dx}"/>
+    <!-- Camera -->
+    <link name="camera_link">
+      <pose>0.2 0 0.3 0 0 0</pose>
+      <visual name="camera_visual">
+        <geometry>
+          <box size="0.05 0.05 0.05"/>
+        </geometry>
+        <xacro:insert_block name="material_white" />
+      </visual>
+    </link>
+    <joint name="camera_joint" type="fixed">
+      <parent link="base_link"/>
+      <child link="camera_link"/>
+      <origin xyz="0.2 0 0.3" rpy="0 0 0"/>
+    </joint>
+    <gazebo reference="camera_link">
+      <sensor name="camera" type="camera">
+        <pose>0 0 0 0 0 0</pose>
+        <visualize>true</visualize>
+        <camera>
+          <horizontal_fov>1.047</horizontal_fov>
+          <image>
+            <width>640</width>
+            <height>480</height>
+            <format>R8G8B8</format>
+          </image>
+          <clip>
+            <near>0.1</near>
+            <far>10</far>
+          </clip>
+          <save enabled="false"/>
+        </camera>
+        <update_rate>30</update_rate>
+        <always_on>true</always_on>
+      </sensor>
+    </gazebo>
   </xacro:macro>
 </robot>
